File: Hardware/pomodoro-pic16f15355/pomodoro.brd (EAGLE design)
At the start: 40 x 67 mm, 33 parts, among them IC1 PIC16F15355T-I_SO

Commit message: Switched out diode and added pchannel mosfet, rounded corners, generated new gergbers
Parts:
- removed D1: CUS10S30,H3F, CUS10S30_H3F:1SS357TPH3F
- added Q1: IRLML2502TRPBF, IRLML2502TRPBF:SOT95P237X112-3N
- added Q2: DMG2305UX-7, DMG2305UX-7:SOT96P240X115-3N
Connections:
- new net N$40: Q1.3, U$2.P$2
- net +3V3: now also Q2.2, U$2.P$1; no longer D1.1
- net GND: now also Q1.2, Q2.1; no longer U$2.P$2
- net N$26: now also Q1.1; no longer U$2.P$1
- net N$41: now also Q2.3; no longer D1.2
Routing:
- net GND: track 298.9 -> 320.0 mm, vias 7 -> 8
- net +3V3: track 104.2 -> 122.1 mm
- net N$26: track 29.1 -> 16.6 mm
- net N$40: track 0.00 -> 5.74 mm
Other:
- outline, holes or cut-outs redrawn
- board text added: "Pomodoro Timer v1.0 RevA"

Commit message: Checked nets Added 3dmodels, moved buzzer to centre and replaced 2mm holes with 3.2mm generated images and gerbers
Parts:
- moved Q2 4.00 mm to (12.5, 3.81)
- moved U$2 1.40 mm to (20.0, 12.3)
- moved Q1 0.92 mm to (25.2, 19.9)
Routing:
- net N$41: track 7.30 -> 12.4 mm
- net N$26: track 16.6 -> 15.6 mm
- net N$40: track 5.74 -> 5.16 mm
- net N$28: track 22.8 -> 22.3 mm
