File: Hardware/pomodoro-py32f002b/pomodoro-py32f002b.sch (EAGLE design)
At the start: 42 parts, among them Q1 IRLML2502TRPBF, Q2 IRLML2502TRPBF, Q3 IRLML2502TRPBF, Q4 DMG2305UX-7

Commit message: Reduce current on sleep by disabling outputs, updated hardware, rounded corners, changed leds from 0805 to 0603
Parts:
- removed Q1, Q2, Q3: IRLML2502TRPBF, IRLML2502TRPBF:IRLML2502TRPBF
- added Q5, Q6, Q7: MMBT3904LT3G, MMBT3904LT3G:MMBT3904LT3G
- added R17: 10K, rcl:R-EU_R0805
- added R18, R4: 10k, rcl:R-EU_R0805
- LEDG1, LEDG2, LEDG3, LEDG4, LEDG5, LEDG6, LEDG7, LEDR1, LEDR2, LEDR3, LEDR4, LEDR5, LEDR6, LEDR7: device led:LEDSML0805 -> SparkFun-LED:LED0603
Connections:
- new net N$16: Q6.B, R4.2
- new net N$19: Q5.B, R18.2
- new net N$6: Q7.B, R17.2
- net BIN: now also R4.1; no longer Q1.G
- net BIN1: now also R17.1; no longer Q2.G
- net GND: now also Q5.E, Q6.E, Q7.E; no longer Q1.S, Q2.S, Q3.S
- net N$10: now also Q7.C; no longer Q2.D
- net N$17: now also Q5.C; no longer Q3.D
- net N$26: now also R18.1; no longer Q3.G
- net N$40: now also Q6.C; no longer Q1.D
Other:
- moved on the sheet: C2, Q4, R10, R11, R12, R13, R14, R15, R9
